Commit message: ultimo robot funcional

File: wamv_description/urdf/wamv_base.urdf.xacro (robot description, xacro)
@@ -26,5 +26,5 @@
    <!-- Center part -->
     <collision name="centerPart">
-      <origin xyz="${0.95-0.6125} 0.0 ${0.5-0.25}"/> <!-- ${0.95-0.4125} -0.085 ${2.95-0.25}" -->
+      <origin xyz="${0.95-0.6125} 0.0 ${0.5-0.25}"/>
       <geometry>
         <box size="0.20 0.5 0.5"/>
@@ -33,7 +33,7 @@
    <!-- Botoom part -->
     <collision name="bottomPart">
-      <origin xyz="0.95 0.0 ${0.5-0.25-0.365}"/> <!--xyz="0.95 -0.085 ${2.95-0.25-0.38} -->
+      <origin xyz="0.95 0.0 ${0.5-0.25-0.365}"/>
       <geometry>
-        <box size="1.3 0.55 0.285"/> <!--size="1.35 0.55 0.285 -->
+        <box size="1.3 0.55 0.285"/>
       </geometry>
     </collision>
@@ -97,6 +97,6 @@
     <inertial>
       <!-- From WAM-V spec sheet -->
-      <mass value="100.0"/>
-      <inertia ixx="120.0" ixy="0.0" ixz="0.0" iyy="393" iyz="0.0" izz="446.0"/>
+      <mass value="180"/>
+      <inertia ixx="120.0" ixy="0.0" ixz="0.0" iyy="393.0" iyz="0.0" izz="446.0"/> <!-- ixx="120.0" ixy="0.0" ixz="0.0" iyy="393" iyz="0.0" izz="446.0" -->
     </inertial>
   </link>

File: wamv_gazebo/urdf/sensors/sonar_sensor.xacro (robot description, xacro)
@@ -3,4 +3,5 @@
 <xacro:macro name="sonar" params="name x y z ros_topic update_rate min_range max_range field_of_view ray_count">
     <joint name="${name}_joint" type="fixed">
+      <origin xyz= "${x} ${y} ${z}" />
       <parent link="base_link"/>
       <child link="${name}_link"/>
@@ -9,17 +10,17 @@
       <inertial>
         <mass value="0.001" />
-        <origin xyz="${x} ${y} ${z}" rpy="0 0 0" />
+        <origin xyz="0 0 0" rpy="0 0 0" />
         <inertia ixx="0.000000017" ixy="0" ixz="0" iyy="0.000000017" iyz="0" izz="0.000000017" />
       </inertial>
       <visual>
-        <origin xyz="${x} ${y} ${z}" rpy="0 0 0" />
+        <origin xyz="0 0 0" rpy="0 0 0" />
         <geometry>
-          <box size="0.01 0.01 0.01" />
+          <box size="0.03 0.03 0.03" />
         </geometry>
       </visual>
       <collision>
-        <origin xyz="${x} ${y} ${z}" rpy="0 0 0" />
+        <origin xyz="0 0 0" rpy="0 0 0" />
         <geometry>
-          <box size="0.01 0.01 0.01" />
+          <box size="0.03 0.03 0.03" />
         </geometry>
       </collision>
@@ -59,4 +60,8 @@
       </sensor>
     </gazebo>
+    <!-- Set color of post -->
+    <gazebo reference="${name}_link">
+      <material>Gazebo/Black</material>
+    </gazebo>
   </xacro:macro>
 </robot>

File: wamv_gazebo/urdf/wamv_gazebo.urdf.xacro (robot description, xacro)
@@ -60,15 +60,18 @@
   <!-- === Sensors === -->
   <!-- Add a stereo camera pair -->
-  <xacro:wamv_camera name="front_left_camera" y="0.1" x="0.75" z="1" P="${radians(15)}" />
-  <xacro:wamv_camera name="front_right_camera" y="-0.1" x="0.75" z="1" P="${radians(15)}" />
-  <xacro:sonar name="sonar_sensor" x="2" y="0" z="2" ros_topic="/distance" update_rate="10" min_range="0.3" max_range="2" field_of_view="56" ray_count="2" />
+  <!-- <xacro:wamv_camera name="front_left_camera"  y="0.1" x="1.5" z="0.65" P="${radians(0)}" /> -->
+  <!-- <xacro:wamv_camera name="front_right_camera" y="-0.1" x="1" z="0.65" P="${radians(15)}" /> -->
+  <xacro:sonar name="sonar_sensor" x="1.6" y="0.4" z="0.6" ros_topic="/distance" update_rate="10" min_range="0.3" max_range="2" field_of_view="56" ray_count="2" />
+  <xacro:sonar name="sonar_sensor2" x="1.6" y="-0.4" z="0.6" ros_topic="/distance2" update_rate="10" min_range="0.3" max_range="2" field_of_view="56" ray_count="2" />
+  <xacro:sonar name="sonar_sensor3" x="0.3" y="0.4" z="0.6" ros_topic="/distance3" update_rate="10" min_range="0.3" max_range="2" field_of_view="56" ray_count="2" />
+  <xacro:sonar name="sonar_sensor4" x="0.3" y="-0.4" z="0.6" ros_topic="/distance4" update_rate="10" min_range="0.3" max_range="2" field_of_view="56" ray_count="2" />
   <!-- Add a camera facing right -->
-  <xacro:wamv_camera name="middle_right_camera" y="0" x="1" z="1" P="${radians(15)}"/> <!-- Y="${radians(-90)}" post_Y="${radians(-90)}" /> -->
+  <xacro:wamv_camera name="middle_right_camera" y="0" x="1.5" z="0.65" P="${radians(50)}"/> <!-- Y="${radians(-90)}" post_Y="${radians(-90)}" /> -->
   <!-- Add simulated GPS -->
-  <xacro:wamv_gps name="gps_wamv" x="-0.85" />
-  <!-- Add Simulated IMU -->
-  <xacro:wamv_imu name="imu_wamv" y="-0.2" />
+  <xacro:wamv_gps name="gps_wamv" x="0.4" y="0" z="0.55"/>
+  <!-- Add Simulated IMU
+  <xacro:wamv_imu name="imu_wamv" y="-0.2" /> -->
   <!-- Add 3D LIDAR -->
-  <xacro:lidar name="lidar_wamv" x="0" y="0" z="2" type="16_beam"/>
+  <xacro:lidar name="lidar_wamv" x="0.8" y="0" z="0.7" type="16_beam"/>
   <!-- Add pinger
   <xacro:wamv_pinger name="pinger" position="1.0 0 -1.0" /> -->
