Commit message: Modificacion de camaras y lidar

File: wamv_gazebo/urdf/sensors/lidar.xacro (robot description, xacro)
@@ -5,7 +5,7 @@
                params = "type:='16_beam'
                          name
-                         x:=0.7 y:=0 z:=1.8
+                         x:=0 y:=0 z:=0
                          R:=0 P:=0 Y:=0
-                         post_Y:=0 post_z_from:=1.2965">
+                         post_Y:=0 post_z_from:=0">
     <xacro:if value="${type == '16_beam'}">
       <xacro:wamv_3d_lidar name="${name}"

File: wamv_gazebo/urdf/sensors/wamv_3d_lidar.xacro (robot description, xacro)
@@ -23,7 +23,7 @@
   -->
   <xacro:macro name="wamv_3d_lidar" params="name
-                                            x:=0.7 y:=0 z:=1.8
+                                            x y z
                                             R:=0 P:=0 Y:=0
-                                            post_Y:=0 post_z_from:=1.2965
+                                            post_Y:=0 post_z_from
                                             update_rate:=10 vertical_lasers:=16 samples:=1875 resolution:=0.1
                                             min_angle:=${-pi} max_angle:=${pi}

File: wamv_gazebo/urdf/sensors/wamv_camera.xacro (robot description, xacro)
@@ -1,5 +1,5 @@
 <?xml version="1.0"?>
 <robot xmlns:xacro="http://ros.org/wiki/xacro">
-  <xacro:macro name="wamv_camera" params="name x:=0.5 y:=0 z:=0.5 post_z_from:=0.5 R:=0 P:=0 Y:=0 post_Y:=0">
+  <xacro:macro name="wamv_camera" params="name x y z post_z_from:=0.2 R:=0 P:=0 Y:=0 post_Y:=0">
     <!-- Define length variables for link positioning -->
     <xacro:property name="platform_z" value="${post_z_from}"/>

File: wamv_gazebo/urdf/sensors/wamv_gps.xacro (robot description, xacro)
@@ -1,8 +1,8 @@
 <?xml version="1.0" encoding="UTF-8"?>
 <robot xmlns:xacro="http://ros.org/wiki/xacro">
-  <xacro:macro name="wamv_gps" params="name:=gps x:=0 y:=0 z:=0.5 R:=0 P:=0 Y:=0 lat:=21.30996 lon:=-157.8901 elev:=0.0 update_rate:=15">
+  <xacro:macro name="wamv_gps" params="name:=gps x y z R:=0 P:=0 Y:=0 lat:=21.30996 lon:=-157.8901 elev:=0.0 update_rate:=15">
     <link name="${name}_link">
       <visual name="${name}_visual">
-        <origin xyz="1.3 0 0"/>
+        <origin xyz="0 0 0"/>
         <geometry>
           <mesh filename="package://wamv_gazebo/models/gps/mesh/gps.dae"/>
@@ -10,5 +10,5 @@
       </visual>
       <collision name="${name}_collision_base">
-        <origin xyz="1 0 0.025" rpy="0 0 0" />
+        <origin xyz="0 0 0" rpy="0 0 0" />
         <geometry>
           <cylinder length="0.05" radius="0.015" />
@@ -16,5 +16,5 @@
       </collision>
       <collision name="${name}_collision_antenna">
-        <origin xyz="0 0 0.11" rpy="0 0 0" />
+        <origin xyz="0 0 0" rpy="0 0 0" />
         <geometry>
           <cylinder length="0.1" radius="0.15" />
