Commit message: remove post from camera

File: wamv_gazebo/urdf/sensors/wamv_camera.xacro (robot description, xacro)
@@ -43,79 +43,10 @@
     <link name="${name}_link_optical">
     </link>
-    <!-- Define post length and mass based on desired z position of sensor -->
-    <xacro:property name="post_length" value="${z-platform_z-post_arm_to_camera_z}"/>
-    <xacro:property name="post_mass_per_meter" value="0.9"/>
-    <xacro:property name="post_mass" value="${post_mass_per_meter * post_length}"/>
-    <xacro:property name="post_radius" value="0.0076"/>
-    <!-- Sensor post -->
-    <link name="${name}_post_link">
-      <visual>
-        <geometry>
-          <cylinder radius="${post_radius}" length="${post_length}"/>
-        </geometry>
-        <material name="${name}_post_material">
-          <color rgba="0.0 0.0 0.0 1.0"/>
-        </material>
-      </visual>
-      <collision name="${name}_post_collision">
-        <geometry>
-          <cylinder radius="${post_radius}" length="${post_length}"/>
-        </geometry>
-      </collision>
-      <inertial>
-        <mass value="${post_mass}"/>
-        <inertia
-          ixx="${(post_mass/12) * (3*post_radius*post_radius + post_length*post_length)}"
-          iyy="${(post_mass/12) * (3*post_radius*post_radius + post_length*post_length)}"
-          izz="${(post_mass/2) * (post_radius*post_radius)}"
-          ixy="0"
-          ixz="0"
-          iyz="0"/>
-      </inertial>
-    </link>
-    <!-- Sensor post arm -->
-    <link name="${name}_post_arm_link">
-      <visual name="${name}_post_arm_visual">
-        <origin xyz="-0.038 0 -0.003" rpy="${radians(-60)} 0 ${-pi/2}"/>
-        <geometry>
-          <mesh filename="package://vrx_gazebo/models/sensor_post/mesh/sensor_post_arm.dae"/>
-        </geometry>
-      </visual>
-      <collision name="${name}_post_arm_collision">
-        <origin xyz="0 0 0" rpy="${radians(-60)-pi/20} 0 ${-pi/2}"/>
-        <geometry>
-          <cylinder radius="0.008" length="0.065"/>
-        </geometry>
-      </collision>
-      <inertial>
-        <origin xyz="0 0 0" rpy="${radians(-60)-pi/20} 0 ${-pi/2}"/>
-        <mass value="0.1"/>
-        <inertia
-          ixx="0.00003680833"
-          iyy="0.00003680833"
-          izz="0.00000320000"
-          ixy="0"
-          ixz="0"
-          iyz="0"/>
-      </inertial>
-    </link>
-    <!-- Base to sensor post joint -->
+    <!-- Base to camera joint -->
     <xacro:property name="post_z" value="${platform_z+post_length/2}"/>
     <xacro:property name="post_to_camera_x" value="${post_to_post_arm_x+post_arm_to_camera_x}"/>
     <joint name="base_to_${name}_post_joint" type="fixed">
-      <origin xyz="${x-(post_to_camera_x)*cos(post_Y)} ${y-(post_to_camera_x)*sin(post_Y)} ${post_z}" rpy="0 0 ${post_Y}" />
+      <origin xyz="${x} ${y} ${z}" rpy="0 0 ${post_Y}" />
       <parent link="base_link" />
-      <child link="${name}_post_link" />
-    </joint>
-    <!-- Sensor post to sensor post arm joint -->
-    <joint name="${name}_post_to_${name}_post_arm_joint" type="fixed">
-      <origin xyz="${post_to_post_arm_x} 0 ${z-post_z-post_arm_to_camera_z}" rpy="0 0 0" />
-      <parent link="${name}_post_link" />
-      <child link="${name}_post_arm_link" />
-    </joint>
-    <!-- Sensor post arm to camera joint -->
-    <joint name="${name}_post_arm_to_${name}_joint" type="fixed">
-      <origin xyz="${post_arm_to_camera_x} 0 ${post_arm_to_camera_z}" rpy="${R} ${P} ${Y-post_Y}" />
-      <parent link="${name}_post_arm_link" />
       <child link="${name}_link" />
     </joint>
