Commit message: add sonar rotation

File: wamv_gazebo/urdf/sensors/sonar_sensor.xacro (robot description, xacro)
@@ -1,5 +1,5 @@
 <?xml version="1.0"?>
 <robot xmlns:xacro="http://ros.org/wiki/xacro">
-<xacro:macro name="sonar" params="name x y z ros_topic update_rate min_range max_range field_of_view ray_count">
+  <xacro:macro name="sonar" params="name x y z R:=0 P:=0 Y:=0 ros_topic update_rate min_range max_range field_of_view ray_count">
     <joint name="${name}_joint" type="fixed">
       <origin xyz= "${x} ${y} ${z}" />
@@ -14,11 +14,11 @@
       </inertial>
       <visual>
-        <origin xyz="0 0 0" rpy="0 0 0" />
+        <origin xyz="0 0 0" rpy="${R} ${P} ${Y}" />
         <geometry>
-          <box size="0.03 0.03 0.03" />
+          <box size="0.1 0.3 0.1" />
         </geometry>
       </visual>
       <collision>
-        <origin xyz="0 0 0" rpy="0 0 0" />
+        <origin xyz="0 0 0" rpy="${R} ${P} ${Y}" />
         <geometry>
           <box size="0.03 0.03 0.03" />
@@ -30,5 +30,5 @@
         <always_on>true</always_on>
         <update_rate>${update_rate}</update_rate>
-        <pose>0 0 0 0 0 0</pose>
+        <pose>0 0 0 ${R} ${P} ${Y}</pose>
         <visualize>false</visualize>
         <ray>

Commit message: sonar: rotacion de los sensores ultrasonicos agregado visual para saber hacia donde esta apuntando

File: wamv_gazebo/urdf/sensors/sonar_sensor.xacro (robot description, xacro)
@@ -3,5 +3,5 @@
   <xacro:macro name="sonar" params="name x y z R:=0 P:=0 Y:=0 ros_topic update_rate min_range max_range field_of_view ray_count">
     <joint name="${name}_joint" type="fixed">
-      <origin xyz= "${x} ${y} ${z}" />
+      <origin xyz= "${x} ${y} ${z}" rpy="${R} ${P} ${Y}" />
       <parent link="base_link"/>
       <child link="${name}_link"/>
@@ -14,13 +14,19 @@
       </inertial>
       <visual>
-        <origin xyz="0 0 0" rpy="${R} ${P} ${Y}" />
+        <origin xyz="0 0 0" rpy="0 0 0" />
         <geometry>
-          <box size="0.1 0.3 0.1" />
+          <box size="0.05 0.05 0.05" />
+        </geometry>
+      </visual>
+      <visual>
+        <origin xyz="0.05 0 0" rpy="0 1.57 ${Y}" />
+        <geometry>
+          <cylinder length="0.06" radius="0.02" />
         </geometry>
       </visual>
       <collision>
-        <origin xyz="0 0 0" rpy="${R} ${P} ${Y}" />
+        <origin xyz="0 0 0" rpy="0 0 0" />
         <geometry>
-          <box size="0.03 0.03 0.03" />
+          <box size="0.05 0.05 0.05" />
         </geometry>
       </collision>
@@ -30,5 +36,5 @@
         <always_on>true</always_on>
         <update_rate>${update_rate}</update_rate>
-        <pose>0 0 0 ${R} ${P} ${Y}</pose>
+        <pose>0 0 0 0 0 0</pose>
         <visualize>false</visualize>
         <ray>

File: wamv_gazebo/urdf/wamv_gazebo.urdf.xacro (robot description, xacro)
@@ -63,8 +63,8 @@
   <!-- <xacro:wamv_camera name="front_right_camera" y="-0.1" x="1" z="0.65" P="${radians(15)}" /> -->
   <xacro:if value="$(arg sonar_enabled)">
-    <xacro:sonar name="sonar_sensor" x="1.6" y="0.4" z="0.6" ros_topic="/distance1" Y="${radians(120)}"  update_rate="10" min_range="0.3" max_range="2" field_of_view="56" ray_count="2" />
-    <xacro:sonar name="sonar_sensor2" x="1.6" y="-0.4" z="0.6" ros_topic="/distance2" update_rate="10" min_range="0.3" max_range="2" field_of_view="56" ray_count="2" />
-    <xacro:sonar name="sonar_sensor3" x="0.3" y="0.4" z="0.6" ros_topic="/distance3" update_rate="10" min_range="0.3" max_range="2" field_of_view="56" ray_count="2" />
-    <xacro:sonar name="sonar_sensor4" x="0.3" y="-0.4" z="0.6" ros_topic="/distance4" Y="${radians(120)}" update_rate="10" min_range="0.3" max_range="2" field_of_view="56" ray_count="2" />
+    <xacro:sonar name="sonar_sensor" x="1.6" y="0.4" z="0.6" ros_topic="/distance1" Y="${radians(0)}"  update_rate="10" min_range="0.3" max_range="2" field_of_view="56" ray_count="2" />
+    <xacro:sonar name="sonar_sensor2" x="1.6" y="-0.4" z="0.6" ros_topic="/distance2" Y="${radians(0)}" update_rate="10" min_range="0.3" max_range="2" field_of_view="56" ray_count="2" />
+    <xacro:sonar name="sonar_sensor3" x="0.3" y="0.4" z="0.6" ros_topic="/distance3" Y="${radians(180)}" update_rate="10" min_range="0.3" max_range="2" field_of_view="56" ray_count="2" />
+    <xacro:sonar name="sonar_sensor4" x="0.3" y="-0.4" z="0.6" ros_topic="/distance4" Y="${radians(180)}" update_rate="10" min_range="0.3" max_range="2" field_of_view="56" ray_count="2" />
   </xacro:if>
   <!-- Add a camera facing right -->
