Commit message: cambios varios

File: wamv_description/urdf/thrusters/engine.xacro (robot description, xacro)
@@ -4,4 +4,5 @@
   <xacro:macro name="engine" params="prefix position:='0 0 0' orientation:='0 0 0'">
     <link name="${prefix}_engine_link">
+      <!--
       <visual>
         <geometry>
@@ -9,4 +10,5 @@
         </geometry>
       </visual>
+      -->
       <collision name="${prefix}_engine_vertical_axis_collision">
         <origin xyz="-0.16 0 -0.24" rpy="0 0 0" />
@@ -33,5 +35,5 @@
       </visual>
       <collision name="${prefix}_propeller_collision">
-        <origin xyz="-0.08 0 0" rpy="0 1.57 0" />
+        <origin xyz="0 0 0" rpy="0 1.57 0" />
         <geometry>
           <cylinder length="0.18" radius="0.24" />

File: wamv_description/urdf/wamv_base.urdf.xacro (robot description, xacro)
@@ -5,5 +5,5 @@
     <!-- Top part -->
     <collision name="topPart">
-      <origin xyz="0.95 -0.085 0.5"/>
+      <origin xyz="0.95 0.0 0.5"/>
       <geometry>
         <box size="1.5 1.1 0.12"/>
@@ -12,5 +12,5 @@
     <!-- External sides -->
     <collision name="${prefix}_externalSide">
-      <origin xyz="${0.95-0.05} ${((0.5-0.06875)*reflect)-0.085} ${0.5-0.29}"/>
+      <origin xyz="${0.95-0.05} ${((0.5-0.06875)*reflect)} ${0.5-0.29}"/>
       <geometry>
         <box size="1.35 0.13 0.67"/>
@@ -19,5 +19,5 @@
     <!-- Internal sides -->
     <collision name="$prefix_internalSide">
-      <origin xyz="${0.95-0.05} ${((0.446875-0.06875-0.065)*reflect)-0.085} ${0.5-0.25}"/>
+      <origin xyz="${0.95-0.05} ${((0.446875-0.06875-0.065)*reflect)} ${0.5-0.25}"/>
       <geometry>
         <box size="1.35 0.15625 0.5"/>
@@ -26,5 +26,5 @@
    <!-- Center part -->
     <collision name="centerPart">
-      <origin xyz="${0.95-0.6125} -0.085 ${0.5-0.25}"/> <!-- ${0.95-0.4125} -0.085 ${2.95-0.25}" -->
+      <origin xyz="${0.95-0.6125} 0.0 ${0.5-0.25}"/> <!-- ${0.95-0.4125} -0.085 ${2.95-0.25}" -->
       <geometry>
         <box size="0.20 0.5 0.5"/>
@@ -33,5 +33,5 @@
    <!-- Botoom part -->
     <collision name="bottomPart">
-      <origin xyz="0.95 -0.085 ${0.5-0.25-0.365}"/> <!--xyz="0.95 -0.085 ${2.95-0.25-0.38} -->
+      <origin xyz="0.95 0.0 ${0.5-0.25-0.365}"/> <!--xyz="0.95 -0.085 ${2.95-0.25-0.38} -->
       <geometry>
         <box size="1.3 0.55 0.285"/> <!--size="1.35 0.55 0.285 -->
@@ -41,5 +41,5 @@
     <!- Top part ->
     <visual>
-      <origin xyz="0.95 -0.085 0.5"/>
+      <origin xyz="0.95 0.0 0.5"/>
       <geometry>
         <box size="1.5 1.1 0.12"/>
@@ -48,5 +48,5 @@
     <!- External sides ->
     <visual>
-      <origin xyz="${0.95-0.05} ${((0.5-0.06875)*reflect)-0.085} ${2.95-0.29}"/>
+      <origin xyz="${0.95-0.05} ${((0.5-0.06875)*reflect)} ${2.95-0.29}"/>
       <geometry>
         <box size="1.35 0.13 0.67"/>
@@ -55,5 +55,5 @@
     <!- Internal sides ->
     <visual>
-      <origin xyz="${0.95-0.05} ${((0.446875-0.06875-0.065)*reflect)-0.085} ${2.95-0.25}"/>
+      <origin xyz="${0.95-0.05} ${((0.446875-0.06875-0.065)*reflect)} ${2.95-0.25}"/>
       <geometry>
         <box size="1.35 0.15625 0.5"/>
@@ -62,5 +62,5 @@
    <!- Center part ->
     <visual>
-      <origin xyz="${0.95-0.6125} -0.085 ${2.95-0.25}"/>
+      <origin xyz="${0.95-0.6125} 0.0 ${2.95-0.25}"/>
       <geometry>
         <box size="0.20 0.5 0.5"/>
@@ -69,5 +69,5 @@
    <!- Botoom part ->
     <visual>
-      <origin xyz="0.95 -0.085 ${2.95-0.25-0.365}"/>
+      <origin xyz="0.95 0.0 ${2.95-0.25-0.365}"/>
       <geometry>
         <box size="1.3 0.55 0.285"/>
@@ -85,5 +85,5 @@
   <link name="dummy_link">
     <visual>
-      <origin xyz="0 0 -0.45" rpy="0 0 0" />
+      <origin xyz="0 0.085 -0.45" rpy="0 0 0" />
       <geometry>
         <mesh filename="package://wamv_description/models/WAM-V-Base/mesh/robot.stl"/>

File: wamv_gazebo/urdf/macros.xacro (robot description, xacro)
@@ -14,3 +14,4 @@
   <xacro:include filename="$(find wamv_gazebo)/urdf/sensors/wamv_p3d.xacro" />
   <xacro:include filename="$(find wamv_gazebo)/urdf/sensors/wamv_pinger.xacro" />
+  <xacro:include filename="$(find wamv_gazebo)/urdf/sensors/sonar_sensor.xacro" />
 </robot>

File: wamv_gazebo/urdf/sensors/wamv_3d_lidar.xacro (robot description, xacro)
@@ -136,5 +136,5 @@
       <child link="${name}_link" />
     </joint>
-    <gazebo reference="${name}_link">
+    <gazebo reference="${namespace}/${name}_link">
       <sensor type="gpu_ray" name="${name}_sensor">
         <update_rate>${update_rate}</update_rate>

File: wamv_gazebo/urdf/sensors/wamv_gps.xacro (robot description, xacro)
@@ -1,7 +1,8 @@
 <?xml version="1.0" encoding="UTF-8"?>
 <robot xmlns:xacro="http://ros.org/wiki/xacro">
-  <xacro:macro name="wamv_gps" params="name:=gps x:=0.3 y:=0 z:=1.3 R:=0 P:=0 Y:=0 lat:=21.30996 lon:=-157.8901 elev:=0.0 update_rate:=15">
+  <xacro:macro name="wamv_gps" params="name:=gps x:=0 y:=0 z:=0.5 R:=0 P:=0 Y:=0 lat:=21.30996 lon:=-157.8901 elev:=0.0 update_rate:=15">
     <link name="${name}_link">
       <visual name="${name}_visual">
+        <origin xyz="1.3 0 0"/>
         <geometry>
           <mesh filename="package://wamv_gazebo/models/gps/mesh/gps.dae"/>
@@ -9,5 +10,5 @@
       </visual>
       <collision name="${name}_collision_base">
-        <origin xyz="0 0 0.025" rpy="0 0 0" />
+        <origin xyz="1 0 0.025" rpy="0 0 0" />
         <geometry>
           <cylinder length="0.05" radius="0.015" />

File: wamv_gazebo/urdf/thruster_layouts/wamv_t_thrusters.xacro (robot description, xacro)
@@ -2,6 +2,7 @@
 <robot xmlns:xacro="http://ros.org/wiki/xacro">
   <xacro:include filename="$(find wamv_description)/urdf/thrusters/engine.xacro" />
-  <xacro:engine prefix="right_rear" position="1 ${-0.085-0.33} 0.318237"  orientation="0.0 0.0 0.0"/> <!-- MID = -0.085--> <!--ori 0.0 0.0 0.785-->
-  <xacro:engine prefix="left_rear" position="1 ${-0.085+0.33} 0.318237" orientation="0.0 0.0 0.0"/> <!--pos 0.5 asd 0.318237 -->
+  <xacro:engine prefix="right" position="${0.95+0.38} ${-0.33} 0.368237"  orientation="0.0 0.0 0.0"/>
+  <xacro:engine prefix="left" position="${0.95+0.38} ${0.33} 0.368237" orientation="0.0 0.0 0.0"/>
+  <xacro:engine prefix="rear" position="${0.68} ${0} 0.265237" orientation="0.0 0.0 0.0"/>
   <!-- <xacro:engine prefix="left_frontt" position="0 1.2  0.25" orientation="0.0 0.0 -0.785"/>
   <xacro:engine prefix="right_frontt" position="0 -1.2 0.25" orientation="0.0 0.0 +0.785"/> -->
@@ -11,8 +12,7 @@
       <robotNamespace>${namespace}</robotNamespace>
       <xacro:include filename="$(find wamv_gazebo)/urdf/thruster_layouts/wamv_gazebo_thruster_config.xacro" />
-      <xacro:wamv_gazebo_thruster_config name="right_rear" />
-      <xacro:wamv_gazebo_thruster_config name="left_rear" />
-      <!--<xacro:wamv_gazebo_thruster_config name="left_frontt" /> -->
-      <!--<xacro:wamv_gazebo_thruster_config name="right_frontt" /> -->
+      <xacro:wamv_gazebo_thruster_config name="right" />
+      <xacro:wamv_gazebo_thruster_config name="left" />
+      <xacro:wamv_gazebo_thruster_config name="rear" />
     </plugin>
   </gazebo>

Commit message: ajustes finales coeficientes dinamicos y flotabilidad

File: wamv_description/urdf/thrusters/engine.xacro (robot description, xacro)
@@ -24,5 +24,5 @@
       </collision>
       <inertial>
-        <mass value="15"/>
+        <mass value="0.1"/>
         <inertia ixx="0.889245" ixy="0.0" ixz="0.0" iyy="0.911125" iyz="0.0" izz="0.078125"/>
       </inertial>
@@ -41,5 +41,5 @@
       </collision>
       <inertial>
-        <mass value="0.5"/>
+        <mass value="0.05"/>
         <inertia ixx="0.008545" ixy="0.0" ixz="0.0" iyy="0.008545" iyz="0.0" izz="0.0144"/>
       </inertial>

File: wamv_description/urdf/wamv_base.urdf.xacro (robot description, xacro)
@@ -39,5 +39,4 @@
     </collision>
 <!-- COLLISIONS VISUALS
-    <!- Top part ->
     <visual>
       <origin xyz="0.95 0.0 0.5"/>
@@ -46,28 +45,24 @@
       </geometry>
     </visual>
-    <!- External sides ->
     <visual>
-      <origin xyz="${0.95-0.05} ${((0.5-0.06875)*reflect)} ${2.95-0.29}"/>
+      <origin xyz="${0.95-0.05} ${((0.5-0.06875)*reflect)} ${0.5-0.29}"/>
       <geometry>
         <box size="1.35 0.13 0.67"/>
       </geometry>
     </visual>
-    <!- Internal sides ->
     <visual>
-      <origin xyz="${0.95-0.05} ${((0.446875-0.06875-0.065)*reflect)} ${2.95-0.25}"/>
+      <origin xyz="${0.95-0.05} ${((0.446875-0.06875-0.065)*reflect)} ${0.5-0.25}"/>
       <geometry>
         <box size="1.35 0.15625 0.5"/>
       </geometry>
     </visual>
-   <!- Center part ->
     <visual>
-      <origin xyz="${0.95-0.6125} 0.0 ${2.95-0.25}"/>
+      <origin xyz="${0.95-0.6125} 0.0 ${0.5-0.25}"/>
       <geometry>
         <box size="0.20 0.5 0.5"/>
       </geometry>
     </visual>
-   <!- Botoom part ->
     <visual>
-      <origin xyz="0.95 0.0 ${2.95-0.25-0.365}"/>
+      <origin xyz="0.95 0.0 ${0.5-0.25-0.365}"/>
       <geometry>
         <box size="1.3 0.55 0.285"/>
@@ -97,6 +92,6 @@
     <inertial>
       <!-- From WAM-V spec sheet -->
-      <mass value="180"/>
-      <inertia ixx="120.0" ixy="0.0" ixz="0.0" iyy="393.0" iyz="0.0" izz="446.0"/> <!-- ixx="120.0" ixy="0.0" ixz="0.0" iyy="393" iyz="0.0" izz="446.0" -->
+      <mass value="16.32"/>
+      <inertia ixx="2.74" ixy="0.0" ixz="0.0" iyy="4.16" iyz="0.0" izz="4.7"/> <!-- ixx="120.0" ixy="0.0" ixz="0.0" iyy="393" iyz="0.0" izz="446.0" -->
     </inertial>
   </link>

File: wamv_gazebo/urdf/dynamics/wamv_gazebo_dynamics_plugin.xacro (robot description, xacro)
@@ -1,5 +1,5 @@
 <?xml version="1.0"?>
 <robot xmlns:xacro="http://ros.org/wiki/xacro">
-  <xacro:macro name="usv_dynamics_gazebo" params="name width:=2.4 length:=4.9">
+  <xacro:macro name="usv_dynamics_gazebo" params="name width:=1.1 length:=1.5">
     <!--Gazebo Plugin for simulating WAM-V dynamics-->
     <gazebo>
@@ -14,16 +14,16 @@
         <nDotR>0.0</nDotR>
         <!-- Linear and quadratic drag -->
-        <xU>51.3</xU>
-        <xUU>72.4</xUU>
-        <yV>40.0</yV>
+        <xU>9.74</xU>
+        <xUU>13.75</xUU>
+        <yV>7.6</yV>
         <yVV>0.0</yVV>
-        <zW>500.0</zW>
-        <kP>50.0</kP>
-        <mQ>50.0</mQ>
-        <nR>400.0</nR>
+        <zW>95</zW>
+        <kP>9.5</kP>
+        <mQ>9.5</mQ>
+        <nR>76</nR>
         <nRR>0.0</nRR>
         <!-- General dimensions -->
         <!--<boatArea>2.2</boatArea>-->
-        <hullRadius>0.213</hullRadius>
+        <hullRadius>0.08</hullRadius>
         <boatWidth>${width}</boatWidth>
         <boatLength>${length}</boatLength>

File: wamv_gazebo/urdf/thruster_layouts/wamv_gazebo_thruster_config.xacro (robot description, xacro)
@@ -13,6 +13,6 @@
       <mappingType>1</mappingType>
       <maxCmd>1.0</maxCmd>
-      <maxForceFwd>250.0</maxForceFwd>
-      <maxForceRev>-100.0</maxForceRev>
+      <maxForceFwd>2.5</maxForceFwd>
+      <maxForceRev>-2.5</maxForceRev>
       <maxAngle>${pi/2}</maxAngle>
     </thruster>
